Commit message: feat: add stage 2 autonomous navigation

File: robocup_home_description/urdf/competition_robot.urdf.xacro (robot description, xacro)
@@ -48,4 +48,11 @@
     </sensor>
   </gazebo>
+  <!-- 仅由 test 模式桥接，用于回归测试统计碰撞；比赛决策禁止订阅此真值。 -->
+  <gazebo reference="base_link">
+    <sensor name="test_base_contact" type="contact">
+      <topic>/test/base_contacts</topic><update_rate>30</update_rate><always_on>true</always_on>
+      <contact><collision>base_link_collision</collision></contact>
+    </sensor>
+  </gazebo>
   <gazebo reference="rgbd_camera_link">
     <sensor name="rgbd_camera" type="rgbd_camera">
